Commit message: apriltag_light

File: vehicles/race.scn.xacro (robot description, xacro)
@@ -98,5 +98,5 @@
             <actuator name="ThrusterSurgePort" type="thruster">
                 <link name="Base"/>
-                <origin rpy="0.0 0.8 -0.52" xyz="-0.86 -0.125 -0.05485"/>
+                <origin rpy="0.0 0.0 -0.52" xyz="-0.86 -0.125 -0.05485"/>
                 <specs thrust_coeff="0.4472" thrust_coeff_backward="0.3566" torque_coeff="0.01" max_rpm="3000.0"/>
                 <propeller diameter="0.08" right="true">
@@ -109,5 +109,5 @@
             <actuator name="ThrusterSurgeStbd" type="thruster">
                 <link name="Base"/>
-                <origin rpy="0.0 0.8 0.52" xyz="-0.86 0.125 -0.05485"/>
+                <origin rpy="0.0 0.0 0.52" xyz="-0.86 0.125 -0.05485"/>
                 <specs thrust_coeff="0.4472" thrust_coeff_backward="0.3566" torque_coeff="0.01" max_rpm="3000.0"/>
                 <propeller diameter="0.08" right="true">
@@ -144,4 +144,10 @@
                 <ros_publisher topic="/${robot_name}/gps/fix"/>
             </sensor>
+            <sensor name="camera_forward" rate="10.0" type="camera">
+                <specs resolution_x="1616" resolution_y="1240" horizontal_fov="60.0"/>
+                <origin rpy="-1.57 3.14 4.71" xyz="0.0 0.0 -0.1767" />
+                <link name="Base"/>
+                <ros_publisher topic="/${robot_name}/camera_forward"/>
+            </sensor>
             <!-- <sensor name="Cam" rate="5.0" type="camera">
                 <link name="Base"/>

File: world/light_apriltag.scn.xacro (robot description, xacro)
@@ -84,5 +84,5 @@
         <world_transform xyz="3.75 -0.5 1.5" rpy="0.0 1.5708 3.1415"/>
     </static>
-    <static name="apriltagsmall_top" type="box">
+    <!-- <static name="apriltagsmall_top" type="box">
         <dimensions xyz="0.05 0.05 0.0001"/>
         <material name="Steel"/>
@@ -107,4 +107,4 @@
         <look name="apriltag13" uv_mode="1"/>
         <world_transform xyz="3.75 -0.25 1.5" rpy="0.0 1.5708 3.1415"/>
-    </static>
+    </static> -->
 </scenario>
